File: hardware/quadcopter.brd (EAGLE design)
At the start: 130.1 x 130.1 mm, 99 parts, among them J1 HEADER-4POS-0.1IN-FEMALE-SMD-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, J2 HEADER-10POSTH-254X10, J3 HEADER-4POS-0.1IN-FEMALE, J4 AVR_SPI_PRG_6-SMD, M1 MOTOR_PADS_GND-MOLEX-SMD, M2 MOTOR_PADS_GND-MOLEX-SMD, M3 MOTOR_PADS_GND-MOLEX-SMD, M4 MOTOR_PADS_GND-MOLEX-SMD, P1 PROPELLOR-45MM, P2 PROPELLOR-45MM, P3 PROPELLOR-45MM, P4 PROPELLOR-45MM, Q1 N-MOSFET-SI2302DS, Q12 N-MOSFET-SI2302DS, Q2 N-MOSFET-SI2302DS, Q3 N-MOSFET-SI2302DS, Q4 N-MOSFET-SI2302DS, Q6 N-MOSFET-SI2302DS, Q8 N-MOSFET-SI2302DS, Q9 N-MOSFET-SI2302DS, SW1 PUSHBUTTON_-4.5X4.5, U1 ATMEGA128RFA1, U2 IMU_LSM9DS1-LSM9DS1, Y1 CRYSTAL5X3

Commit message: Updated IMU pads and aligned parts to 0.5mm grid
Parts:
- moved D17 0.80 mm to (-36.0, -14.0)
- moved SW1 0.75 mm to (7.00, -10.0)
- moved J4 0.59 mm to (-16.0, 2.50)
- moved VR1 0.41 mm to (-10.5, -10.5)
- moved J1 0.35 mm to (-25.0, 3.00)
- moved J2 0.13 mm to (-12.5, -5.00)
Routing:
- net 2V5: track 65.4 -> 69.5 mm, vias 13 -> 11
- net RESET: track 55.7 -> 57.3 mm
- net MISO: track 43.6 -> 45.1 mm
- net N$24: track 4.08 -> 4.89 mm
- net SCK: track 43.9 -> 44.4 mm
